File: ZXCT210.kicad_sch (KiCad schematic)
At the start: 6 parts, among them U1 ZXCT210

Commit message: Add files via upload
Parts:
- added R2: {ROUT}, symbol ZXCT210:R
- added U2: CEU4J2X7R2A103K125AE_s, symbol ZXCT210:C
Connections:
- net 0: now also U2.2
- net OUT: now also R2.2, U2.1; no longer U1.6 (OUT)
- new net CNV: R2.1, U1.6 (OUT)
Other:
- note added: "VOUT = ((ILOAD * RSENSE)* GAIN) + VREF"
- moved on the sheet: I1
